Commit message: project 2 updates

File: project2/catkin_ws/src/my_robot/urdf/my_robot.xacro (robot description, xacro)
@@ -160,4 +160,36 @@
     <material>Gazebo/Red</material>
   </gazebo>
+  <link name='camera_rear'>
+    <inertial>
+      <mass value="0.1"/>
+      <origin xyz="0 0 0" rpy=" 0 0 0"/>
+      <inertia
+          ixx="1e-6" ixy="0" ixz="0"
+          iyy="1e-6" iyz="0"
+          izz="1e-6"
+      />
+    </inertial>
+    <collision name='collision'>
+      <origin xyz="0 0 0" rpy=" 0 0 0"/>
+      <geometry>
+        <box size="0.05 0.05 0.05"/>
+      </geometry>
+    </collision>
+    <visual name='camera_rear'>
+      <origin xyz="0 0 0" rpy=" 0 0 0"/>
+      <geometry>
+        <box size="0.05 0.05 0.05"/>
+      </geometry>
+    </visual>
+  </link>
+  <joint type="fixed" name="camera_rear_joint">
+    <origin xyz="-0.2 0 0" rpy=" 0 0 3.14159"/>
+    <axis xyz="1 0 0" rpy=" 0 0 0"/>
+    <parent link='chassis'/>
+    <child link='camera_rear'/>
+  </joint>
+  <gazebo reference="camera_rear">
+    <material>Gazebo/Red</material>
+  </gazebo>
   <link name='hokuyo'>
     <inertial>
